File: board/v0.2/decelerator4030.sch (KiCad schematic (older format))
At the start: 67 parts, among them CON1 A3000/A4000_LOCAL_BUS_SLOT, J3 XILINX_JTAG, J4 CONN_2, J5 CONN_4, U1 MC68030FE, U10 74LXC245, U11 74LXC245, U12 MCP9801, U13 DS1086L, U14 XTAL_OSC_DIP8, U15 MCP1826S, U16 IS66WVE4M16, U17 IS66WVE4M16, U18 MC68030FE_PGA, U2 XC95144XL-10TQG144C, U3 AS6C3216, U4 AS6C3216, U5 S29AL016J, U6 S29AL016J, U7 PCA9564, U8 74LXC245, U9 74LXC245

Commit message: New version schematic and board
Parts:
- added C30, C31, C32: 100nF, ~, symbol C
- added U19: XC9536XL-5VQG44C, ~, symbol XC9536XL-5VQG44C
- U18: value MC68030FE_PGA -> MC68030RC_PGA
Connections:
- net +3.3V: now also C30.1, C31.1, C32.1, U19.15 (VCCINT), U19.26 (VCCIO), U19.35 (VCCINT)
- net 68030CLK: now also U19.44 (IO1-5/GCK2)
- net A19: now also U19.5 (IO1-9)
- net A20: now also U19.6 (IO1-10)
- net A21: now also U19.7 (IO1-11)
- net A22: now also U19.8 (IO1-12)
- net A23: now also U19.12 (IO1-13)
- net A24: now also U19.13 (IO1-14); no longer U2.68 (IO5-10)
- net A25: now also U19.14 (IO1-15); no longer U2.58 (IO5-11)
- net A26: now also U19.16 (IO1-16); no longer U2.60 (IO5-12)
- net A27: now also U19.18 (IO1-17)
- net A28: now also U19.19 (IO2-17)
- net A29: now also U19.20 (IO2-16)
- net A30: now also U19.21 (IO2-15)
- net A31: now also U19.22 (IO2-14)
- net D24: now also U2.133 (IO4-3)
- net D25: now also U2.134 (IO4-12)
- net D26: now also U2.135 (IO4-10)
- net D27: now also U2.136 (IO4-14)
- net GND: now also C30.2, C31.2, C32.2, U19.17 (GND), U19.25 (GND), U19.4 (GND)
- net LOGIC_CLK: now also U19.43 (IO1-3/GCK1)
- net MA24: now also U2.68 (IO5-10), U19.3 (IO1-8); no longer U2.26 (IO1-12)
- net MA25: now also U2.58 (IO5-11), U19.2 (IO1-6); no longer U2.27 (IO1-14)
- net MA26: now also U2.60 (IO5-12), U19.1 (IO1-7/GCK3); no longer U2.28 (IO1-15)
- net R_W: now also U2.23 (IO1-1), U19.41 (IO1-2); no longer U2.136 (IO4-14)
- net SIZ0: now also U2.142 (IO2-1); no longer U2.143 (IO2-2/GSR)
- net _AS: now also CON1.133 (_AS), U19.40 (IO1-1)
- net _BGACK: now also U19.42 (IO1-4)
- net _BG_QFP: now also U2.126 (IO4-2); no longer U2.133 (IO4-3)
- net _DS: now also CON1.97 (_DS)
- net _ECS: now also U2.24 (IO1-11), U19.38 (IO2-2); no longer U2.142 (IO2-1)
- net _OCS: now also U2.27 (IO1-14); no longer U2.134 (IO4-12)
- net _RESET: now also U2.143 (IO2-2/GSR), U19.33 (IO2-6/GSR); no longer U2.135 (IO4-10)
- net TDO1: now reaches U2.122 (TDO)
- net TDO1: now also U19.9 (TDI); no longer J3.3 (TDO)
- net TMS: now reaches J3.1 (TMS), U2.65 (TMS)
- net TMS: now also U19.10 (TMS)
- net TCK: now reaches J3.4 (TCK), U2.67 (TCK)
- net TCK: now also U19.11 (TCK)
- removed net _MAS: CON1.133 (_AS), U2.23 (IO1-1)
- removed net _MDS: CON1.97 (_DS), U2.24 (IO1-11)
- new net TDO2: J3.3 (TDO), U19.24 (TDO)
- new net _MAPEN: U19.39 (IO2-1), U2.28 (IO1-15)
Other:
- moved on the sheet: C16, C17, C18, C19, C20, C7, J5, JP4, JP5, R3, U15

Commit message: Some change boards and schematic
Connections:
- net 3.3V is gone; now on net +3.3V: C7.2, U15.3 (VOUT)
- net +5V: now also C27.1, C28.1, C29.1, U18.C6 (VCC), U18.D10 (VCC), U18.D4 (VCC), U18.F11 (VCC), U18.F2 (VCC), U18.H11 (VCC), U18.H3 (VCC), U18.K10 (VCC), U18.K4 (VCC), U18.L6 (VCC); no longer CON1.176 (D1), CON1.180 (D2), CON1.184 (D3), U1.76 (D1), U1.78 (D2), U1.79 (D3), U18.K12 (D1), U18.L13 (D2), U18.M13 (D3), U8.12 (B6), U8.13 (B5), U8.14 (B4)
- net A10: now also U2.70 (IO5-13); no longer U2.40 (IO3-9)
- net A11: now also U2.57 (IO5-9); no longer U2.48 (IO3-10)
- net A12: now also U2.61 (IO5-14); no longer U2.43 (IO3-11)
- net A13: now also U2.68 (IO5-10); no longer U2.45 (IO3-12)
- net A14: now also U2.58 (IO5-11); no longer U2.49 (IO3-14)
- net A15: now also U2.64 (IO5-15); no longer U2.50 (IO3-15)
- net A16: now also U2.54 (IO5-6); no longer U2.51 (IO3-17)
- net A17: now also U2.59 (IO5-3); no longer U2.52 (IO5-2)
- net A18: now also U2.51 (IO3-17); no longer U2.59 (IO5-3)
- net A19: now also U19.22 (IO2-14), U2.56 (IO5-8); no longer U19.5 (IO1-9), U2.53 (IO5-5)
- net A20: now also U19.21 (IO2-15), U2.53 (IO5-5); no longer U19.6 (IO1-10), U2.54 (IO5-6)
- net A21: now also U19.20 (IO2-16), U2.52 (IO5-2); no longer U19.7 (IO1-11), U2.66 (IO5-7)
- net A22: now also U19.19 (IO2-17), U2.50 (IO3-15); no longer U19.8 (IO1-12), U2.56 (IO5-8)
- net A23: now also U19.18 (IO1-17), U2.49 (IO3-14); no longer U19.12 (IO1-13), U2.57 (IO5-9)
- net A24: now also U19.16 (IO1-16); no longer U19.13 (IO1-14)
- net A26: now also U19.13 (IO1-14); no longer U19.16 (IO1-16)
- net A27: now also U19.12 (IO1-13), U2.48 (IO3-10); no longer U19.18 (IO1-17), U2.70 (IO5-13)
- net A28: now also U19.8 (IO1-12), U2.46 (IO3-7); no longer U19.19 (IO2-17), U2.61 (IO5-14)
- net A29: now also U19.7 (IO1-11), U2.45 (IO3-12); no longer U19.20 (IO2-16), U2.64 (IO5-15)
- net A30: now also U19.6 (IO1-10), U2.44 (IO3-4); no longer U19.21 (IO2-15), U2.69 (IO5-17)
- net A31: now also U19.5 (IO1-9), U2.43 (IO3-11); no longer U19.22 (IO2-14), U2.71 (IO7-2)
- net A4: now also U2.71 (IO7-2); no longer U2.39 (IO3-1)
- net A5: now also U2.69 (IO5-17); no longer U2.41 (IO3-3)
- net A6: now also U2.66 (IO5-7); no longer U2.44 (IO3-4)
- net A9: now also U2.60 (IO5-12); no longer U2.46 (IO3-7)
- net MA24: now also U2.39 (IO3-1); no longer U2.68 (IO5-10)
- net MA25: now also U2.40 (IO3-9); no longer U2.58 (IO5-11)
- net MA26: now also U2.41 (IO3-3); no longer U2.60 (IO5-12)
- net _I2CCE: now also U2.124 (IO6-15); no longer U2.125 (IO6-17)
- net _I2CINT: now also U2.125 (IO6-17); no longer U2.124 (IO6-15)
- new net D1: CON1.176 (D1), U1.76 (D1), U18.K12 (D1), U8.12 (B6)
- new net D2: CON1.180 (D2), U1.78 (D2), U18.L13 (D2), U8.13 (B5)
- new net D3: CON1.184 (D3), U1.79 (D3), U18.M13 (D3), U8.14 (B4)
Changed lines of the file:
@@
 Sheet 1 1
 Title "Decelerator4030"
-Date "21 oct 2014"
+Date "4 nov 2014"
 Rev "0.2"
 Comp ""
@@
 	3100 6350 3200 6450
 Entry Wire Line
-	3200 6350 3300 6450
-Entry Wire Line
 	3400 6350 3500 6450
 Entry Wire Line
@@
 	3700 6350 3800 6450
 Entry Wire Line
-	3800 6350 3900 6450
-Entry Wire Line
-	4000 6350 4100 6450
-Entry Wire Line
 	4200 6350 4300 6450
 Entry Wire Line
@@
 	0    -1   -1   0
 $EndComp
-Text GLabel 3300 6250 1    39   Input ~ 0
+Text GLabel 3350 6250 1    39   Input ~ 0
 68030CLK
-Text GLabel 4600 10200 3    39   Output ~ 0
+Text GLabel 4800 10200 3    39   Output ~ 0
 _I2CCE
 Text GLabel 6200 6250 1    39   Input ~ 0
@@
 Text GLabel 18050 2250 2    39   Input ~ 0
 _I2CWR
-Text GLabel 4800 10200 3    39   Input ~ 0
+Text GLabel 4600 10200 3    39   Input ~ 0
 _I2CINT
 Text GLabel 4900 10200 3    39   Output ~ 0
@@
 	1    0    0    -1
 $EndComp
-Text GLabel 22600 6100 2    39   Output ~ 0
-3.3V
 $Comp
 L +5V #PWR037
@@
 Text Label 4300 6500 1    59   ~ 0
 A3
-Text Label 4100 6500 1    59   ~ 0
+Text Label 4100 9900 1    59   ~ 0
 A4
-Text Label 3900 6500 1    59   ~ 0
+Text Label 6000 9950 1    59   ~ 0
 A5
-Text Label 3800 6500 1    59   ~ 0
+Text Label 6900 9950 1    59   ~ 0
 A6
 Text Label 3700 6500 1    59   ~ 0
@@
 Text Label 3600 6500 1    59   ~ 0
 A8
-Text Label 3500 6500 1    59   ~ 0
+Text Label 6400 9950 1    59   ~ 0
 A9
-Text Label 3300 6500 1    59   ~ 0
+Text Label 6300 9950 1    59   ~ 0
 A10
-Text Label 3200 6500 1    59   ~ 0
+Text Label 6700 9950 1    59   ~ 0
 A11
-Text Label 3100 6500 1    59   ~ 0
+Text Label 6200 9950 1    59   ~ 0
 A12
-Text Label 3000 6500 1    59   ~ 0
+Text Label 6600 9950 1    59   ~ 0
 A13
-Text Label 2900 6500 1    59   ~ 0
+Text Label 6500 9950 1    59   ~ 0
 A14
-Text Label 2800 6500 1    59   ~ 0
+Text Label 6100 9950 1    59   ~ 0
 A15
-Text Label 2700 6500 1    59   ~ 0
+Text Label 7000 9950 1    59   ~ 0
 A16
-Text Label 7300 9950 1    59   ~ 0
-A17
 Text Label 7200 9950 1    59   ~ 0
+A17
+Text Label 2700 6500 1    59   ~ 0
 A18
-Text Label 7100 9950 1    59   ~ 0
+Text Label 6800 9950 1    59   ~ 0
 A19
-Text Label 7000 9950 1    59   ~ 0
+Text Label 7100 9950 1    59   ~ 0
 A20
-Text Label 6900 9950 1    59   ~ 0
+Text Label 7300 9950 1    59   ~ 0
 A21
-Text Label 6800 9950 1    59   ~ 0
+Text Label 2800 6500 1    59   ~ 0
 A22
-Text Label 6700 9950 1    59   ~ 0
+Text Label 2900 6500 1    59   ~ 0
 A23
-Text Label 6300 9950 1    59   ~ 0
+Text Label 3200 6500 1    59   ~ 0
 A27
-Text Label 6200 9950 1    59   ~ 0
+Text Label 3500 6500 1    59   ~ 0
 A28
-Text Label 6100 9950 1    59   ~ 0
+Text Label 3000 6500 1    59   ~ 0
 A29
-Text Label 6000 9950 1    59   ~ 0
+Text Label 3800 6500 1    59   ~ 0
 A30
-Text Label 4100 9950 1    59   ~ 0
+Text Label 3100 6500 1    59   ~ 0
 A31
 Text Label 12050 10050 1    59   ~ 0
@@
 Text Label 14800 2250 1    59   ~ 0
 D4
-Text Label 14500 2250 1    59   ~ 0
+Text Label 14500 2200 1    59   ~ 0
 D3
-Text Label 14200 2250 1    59   ~ 0
+Text Label 14200 2200 1    59   ~ 0
 D2
-Text Label 13900 2250 1    59   ~ 0
+Text Label 13900 2200 1    59   ~ 0
 D1
 Text Label 13600 2250 1    59   ~ 0
@@
 	3200 6550 3200 6450
 Wire Wire Line
-	3300 6450 3300 6550
-Wire Wire Line
 	3500 6450 3500 6550
 Wire Wire Line
@@
 	3800 6550 3800 6450
 Wire Wire Line
-	3900 6450 3900 6550
-Wire Wire Line
-	4100 6550 4100 6450
-Wire Wire Line
 	4300 6450 4300 6550
 Wire Wire Line
@@
 	20250 3350 20600 3350
 Wire Wire Line
-	3300 6250 3300 6400
-Wire Wire Line
-	3300 6400 3400 6400
-Wire Wire Line
 	3400 6400 3400 6550
 Wire Bus Line
@@
 Connection ~ 16250 8000
 Wire Wire Line
-	16250 7700 16250 9800
+	16250 7750 16250 9800
 Wire Wire Line
 	16500 8100 16250 8100
@@
 Wire Wire Line
 	21550 13950 21550 13700
-Text Label 19400 12600 0    39   ~ 0
+Text Label 21550 13850 1    39   ~ 0
 A19
-Text Label 19400 12700 0    39   ~ 0
+Text Label 21450 13850 1    39   ~ 0
 A20
-Text Label 19400 12800 0    39   ~ 0
+Text Label 21350 13850 1    39   ~ 0
 A21
-Text Label 19400 12900 0    39   ~ 0
+Text Label 21250 13850 1    39   ~ 0
 A22
-Text Label 20550 13850 1    39   ~ 0
+Text Label 21150 13850 1    39   ~ 0
 A23
-Text Label 20650 13850 1    39   ~ 0
+Text Label 20950 13850 1    39   ~ 0
 A24
 Text Label 20750 13850 1    39   ~ 0
 A25
-Text Label 20950 13850 1    39   ~ 0
+Text Label 20650 13850 1    39   ~ 0
 A26
-Text Label 21150 13850 1    39   ~ 0
+Text Label 20550 13850 1    39   ~ 0
 A27
-Text Label 21250 13850 1    39   ~ 0
+Text Label 19400 12900 0    39   ~ 0
 A28
-Text Label 21350 13850 1    39   ~ 0
+Text Label 19400 12800 0    39   ~ 0
 A29
-Text Label 21450 13850 1    39   ~ 0
+Text Label 19400 12700 0    39   ~ 0
 A30
-Text Label 21550 13850 1    39   ~ 0
+Text Label 19400 12600 0    39   ~ 0
 A31
 Text GLabel 7950 8750 2    39   Output ~ 0
@@
 Wire Wire Line
 	21750 14750 22250 14750
-Text GLabel 6450 10200 3    39   BiDi ~ 0
+Text GLabel 3850 6250 1    39   BiDi ~ 0
 MA26
-Text GLabel 6550 10200 3    39   BiDi ~ 0
+Text GLabel 3250 6250 1    39   BiDi ~ 0
 MA25
-Text GLabel 6650 10200 3    39   BiDi ~ 0
+Text GLabel 4050 6250 1    39   BiDi ~ 0
 MA24
 Wire Wire Line
-	6450 10200 6450 9950
-Wire Wire Line
-	6450 9950 6400 9950
-Wire Wire Line
 	6400 9950 6400 9750
 Wire Wire Line
-	6550 10200 6550 9950
-Wire Wire Line
-	6550 9950 6500 9950
-Wire Wire Line
 	6500 9950 6500 9750
 Wire Wire Line
 	6600 9750 6600 9950
-Wire Wire Line
-	6600 9950 6650 9950
-Wire Wire Line
-	6650 9950 6650 10200
 Text GLabel 21150 11250 1    39   Input ~ 0
 _ECS
 Wire Wire Line
 	21150 11250 21150 11600
+$Comp
+L +3.3V #PWR078
+U 1 1 54569FF3
+P 22600 6100
+F 0 "#PWR078" H 22600 6060 30  0001 C CNN
+F 1 "+3.3V" H 22600 6210 30  0000 C CNN
+F 2 "" H 22600 6100 60  0000 C CNN
+F 3 "" H 22600 6100 60  0000 C CNN
+	1    22600 6100
+	0    1    1    0
+$EndComp
+Wire Wire Line
+	4100 6550 4100 6450
+Wire Wire Line
+	4100 6450 4050 6450
+Wire Wire Line
+	4050 6450 4050 6250
+Wire Wire Line
+	3400 6400 3350 6400
+Wire Wire Line
+	3350 6400 3350 6250
+Wire Wire Line
+	3300 6550 3300 6400
+Wire Wire Line
+	3300 6400 3250 6400
+Wire Wire Line
+	3250 6400 3250 6250
+Wire Wire Line
+	3900 6550 3900 6450
+Wire Wire Line
+	3900 6450 3850 6450
+Wire Wire Line
+	3850 6450 3850 6250
+Entry Wire Line
+	6400 9950 6500 10050
+Entry Wire Line
+	6500 9950 6600 10050
+Entry Wire Line
+	6600 9950 6700 10050
 $EndSCHEMATC

Commit message: semifinal board prototype
Parts:
- added C33, C34, C35, C36, C37, C38, C39: 100nF, ~, symbol C
- added U20: MCP9801, symbol MCP9801
Connections:
- net +3.3V: now also U13.5 (OE), U13.6 (PDN), C33.2, C34.1, C35.1, C36.1, C37.1, C38.1, C39.1, U20.5 (A2), U20.8 (VDD)
- net ARM0: now also U16.C4 (A6), U17.C4 (A6); no longer U16.A3 (A0), U17.A3 (A0)
- net ARM1: now also U16.A5 (A2), U17.A5 (A2); no longer U16.A4 (A1), U17.A4 (A1)
- net ARM10: now also U16.G3 (A12), U17.G3 (A12); no longer U16.H4 (A10), U17.H4 (A10)
- net ARM11: now also U16.H3 (A9), U17.H3 (A9); no longer U16.H5 (A11), U17.H5 (A11)
- net ARM12: now also U16.E4 (A16), U17.E4 (A16); no longer U16.G3 (A12), U17.G3 (A12)
- net ARM13: now also U16.H4 (A10), U17.H4 (A10); no longer U16.G4 (A13), U17.G4 (A13)
- net ARM14: now also U16.G4 (A13), U17.G4 (A13); no longer U16.F3 (A14), U17.F3 (A14)
- net ARM15: now also U16.H5 (A11), U17.H5 (A11); no longer U16.F4 (A15), U17.F4 (A15)
- net ARM16: now also U16.H6 (A20), U17.H6 (A20); no longer U16.E4 (A16), U17.E4 (A16)
- net ARM17: now also U16.E3 (A21), U17.E3 (A21); no longer U16.D3 (A17), U17.D3 (A17)
- net ARM18: now also U16.G2 (A19), U17.G2 (A19); no longer U16.H1 (A18), U17.H1 (A18)
- net ARM19: now also U16.H1 (A18), U17.H1 (A18); no longer U16.G2 (A19), U17.G2 (A19)
- net ARM2: now also U16.B4 (A4), U17.B4 (A4); no longer U16.A5 (A2), U17.A5 (A2)
- net ARM20: now also U16.F4 (A15), U17.F4 (A15); no longer U16.H6 (A20), U17.H6 (A20)
- net ARM21: now also U16.D4 (A7), U17.D4 (A7); no longer U16.E3 (A21), U17.E3 (A21)
- net ARM3: now also U16.A4 (A1), U17.A4 (A1); no longer U16.B3 (A3), U17.B3 (A3)
- net ARM4: now also U16.D3 (A17), U17.D3 (A17); no longer U16.B4 (A4), U17.B4 (A4)
- net ARM5: now also U16.A3 (A0), U17.A3 (A0); no longer U16.C3 (A5), U17.C3 (A5)
- net ARM6: now also U16.B3 (A3), U17.B3 (A3); no longer U16.C4 (A6), U17.C4 (A6)
- net ARM7: now also U16.C3 (A5), U17.C3 (A5); no longer U16.D4 (A7), U17.D4 (A7)
- net ARM8: now also U16.F3 (A14), U17.F3 (A14); no longer U16.H2 (A8), U17.H2 (A8)
- net ARM9: now also U16.H2 (A8), U17.H2 (A8); no longer U16.H3 (A9), U17.H3 (A9)
- net DRM10: now also U16.C1 (DQ9); no longer U16.C2 (DQ10)
- net DRM13: now also U16.F1 (DQ14); no longer U16.F2 (DQ13)
- net DRM14: now also U16.F2 (DQ13); no longer U16.F1 (DQ14)
- net DRM21: now also U17.F6 (DQ6); no longer U17.F5 (DQ5)
- net DRM22: now also U17.F5 (DQ5); no longer U17.F6 (DQ6)
- net DRM25: now also U17.C2 (DQ10); no longer U17.C1 (DQ9)
- net DRM26: now also U17.C1 (DQ9); no longer U17.C2 (DQ10)
- net DRM29: now also U17.F1 (DQ14); no longer U17.F2 (DQ13)
- net DRM30: now also U17.F2 (DQ13); no longer U17.F1 (DQ14)
- net DRM5: now also U16.F6 (DQ6); no longer U16.F5 (DQ5)
- net DRM6: now also U16.F5 (DQ5); no longer U16.F6 (DQ6)
- net DRM9: now also U16.C2 (DQ10); no longer U16.C1 (DQ9)
- net GND: now also C33.1, C34.2, C35.2, C36.2, C37.2, C38.2, C39.2, U20.4 (GND), U20.6 (A1), U20.7 (A0)
- net SCL: now also U20.2 (SCL)
- net SDA: now also U20.1 (SDA)
- net at R6.1, U12.3 (ALRT): now also U20.3 (ALRT)
