File: board/v0.2/decelerator4030.sch (KiCad schematic (older format))
At the start: 81 parts, among them CON1 A3000/A4000_LOCAL_BUS_SLOT, J3 XILINX_JTAG, J4 CONN_2, J5 CONN_4, U1 MC68030FE, U10 74LXC245, U11 74LXC245, U12 MCP9801, U13 DS1086L, U14 XTAL_OSC_DIP8, U15 MCP1826S, U16 IS66WVE4M16, U17 IS66WVE4M16, U18 MC68030RC_PGA, U19 XC9536XL-5VQG44C, U2 XC95144XL-10TQG144C, U20 MCP9801, U3 AS6C3216, U4 AS6C3216, U5 S29AL016J, U6 S29AL016J, U7 PCA9564, U8 74LXC245, U9 74LXC245

Commit message: Revert "Final proto board and gerber files"
This reverts commit 2b0c9fd41709aa66afef538672b8e5c53e5a6036.
Parts:
- removed C40, C41: 1uF, ~, symbol C
