File: board/v0.2/decelerator4030.kicad_pcb (KiCad board)
At the start: 2 copper layers, 174 parts, among them CON1 A3000/A4000_LOCAL_BUS_SLOT, J3 XILINX_JTAG, J4 CONN_2, J5 CONN_4, U1 MC68030FE, U10 74LXC245, U11 74LXC245, U12 MCP9801, U13 DS1086L, U14 XTAL_OSC_DIP8, U15 MCP1826S, U16 IS66WVE4M16, U17 IS66WVE4M16, U18 MC68030RC_PGA, U19 XC9536XL-5VQG44C, U2 XC95144XL-10TQG144C, U20 MCP9801, U3 AS6C3216, U4 AS6C3216, U5 S29AL016J, U6 S29AL016J, U7 PCA9564, U8 74LXC245, U9 74LXC245

Commit message: Revert "Final proto board and gerber files"
This reverts commit 2b0c9fd41709aa66afef538672b8e5c53e5a6036.
Parts:
- removed ? (x89): , PINTST_0.5
- removed C40, C41: 1uF, SM1210L
- removed Hole_4mm (x4): P***, hole_4mm
- moved C31 1.28 mm to (44.6, 97.3)
- moved C30 1.24 mm to (48.2, 107.7)
- moved C32 1.16 mm to (53.0, 92.2)
- moved U19 1.12 mm to (52.3, 99.7)
Routing:
- net GND: track 695.8 -> 747.1 mm, vias 112 -> 114
- net /DRM15: track 85.4 -> 69.0 mm
- net /DRM14: track 88.3 -> 72.9 mm
- net /DRM13: track 85.5 -> 73.0 mm
- net +3.3V: track 812.4 -> 800.1 mm
- net /DRM12: track 87.2 -> 75.4 mm
- net _RESET_CPLD: track 93.5 -> 83.6 mm
- net /DRM11: track 85.5 -> 75.7 mm
- net _FLASH_WE: track 99.7 -> 90.6 mm
- net /DRM10: track 82.6 -> 74.5 mm
- net _IDBUS_UUB: track 116.1 -> 108.2 mm
- net _FLASH_BUSY: track 102.4 -> 94.8 mm
- net /DRM24: track 111.3 -> 104.8 mm
- net /DRM9: track 84.1 -> 77.9 mm
- net (no net): track 16.7 -> 10.5 mm, vias 4 -> 1
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Other:
- board text removed: "By: strim_ jarob asman"
- board text removed: "Decelerator 4030 Proto v1.0"
- board text removed: "SAKURA"
